File: sumo_tennsy.sch (KiCad schematic (older format))
At the start: 42 parts, among them J1 CONN_01X03, J10 TB_1X2, J11 TB_1X2, J12 HEADER_2, J13 HEADER_2, J14 TB_1X2, J15 HEADER_2, J16 HEADER_2, J17 CONN_01X03, J2 CONN_01X03, J3 CONN_01X03, J4 CONN_01X03, J5 CONN_01X03, J6 CONN_01X03, J7 CONN_01X03, J8 CONN_01X03, J9 HEADER_4, P1 HEADER_02X05, P2 HEADER_02X05, Q1 2N7002, U1 Teensy4.0, U2 MCP2515-xSO, U3 TJA1050, U4 LM1117-SOT

Commit message: modifcaciones
se agrego vista 3d y se modifico pcb
Parts:
- Brd1: symbol SSD1306-128x64_OLED:SSD1306 -> sumo_tennsy-rescue:SSD1306-SSD1306-128x64_OLED
- D1, D2: symbol LED:WS2812B -> sumo_tennsy-rescue:WS2812B-LED
Other:
- moved on the sheet: Brd1, C3, C4, C5, LED1, R3
Changed lines of the file:
@@
 EESchema Schematic File Version 4
+LIBS:sumo_tennsy-cache
 EELAYER 30 0
 EELAYER END
@@
 $EndComp
 $Comp
-L LED:WS2812B D1
+L sumo_tennsy-rescue:WS2812B-LED D1
 U 1 1 5FCE0D89
 P 8200 1150
@@
 $EndComp
 $Comp
-L LED:WS2812B D2
+L sumo_tennsy-rescue:WS2812B-LED D2
 U 1 1 5FCE22F5
 P 9100 1150
@@
 A7
 $Comp
-L SSD1306-128x64_OLED:SSD1306 Brd1
+L sumo_tennsy-rescue:SSD1306-SSD1306-128x64_OLED Brd1
 U 1 1 5FD406EA
-P 5150 2050
-F 0 "Brd1" H 4872 2062 50  0000 R CNN
-F 1 "SSD1306" H 4872 2153 50  0000 R CNN
-F 2 "SSD1306:128x64OLED" H 5150 2300 50  0001 C CNN
-F 3 "" H 5150 2300 50  0001 C CNN
-	1    5150 2050
+P 4900 1200
+F 0 "Brd1" H 4622 1212 50  0000 R CNN
+F 1 "SSD1306" H 4622 1303 50  0000 R CNN
+F 2 "SSD1306:128x64OLED" H 4900 1450 50  0001 C CNN
+F 3 "" H 4900 1450 50  0001 C CNN
+	1    4900 1200
 	-1   0    0    1
 $EndComp
 Wire Wire Line
-	5000 2400 5000 2550
+	4750 1550 4750 1700
 Wire Wire Line
-	5000 2550 4800 2550
+	4750 1700 4550 1700
 Wire Wire Line
-	4800 2650 5100 2650
+	4550 1800 4850 1800
 Wire Wire Line
-	5100 2650 5100 2400
+	4850 1800 4850 1550
 Wire Wire Line
-	5200 2650 5600 2650
+	4950 1800 5350 1800
 Wire Wire Line
-	5600 2650 5600 1700
+	5350 1800 5350 850
 Wire Wire Line
-	5300 2400 5300 2850
+	5050 1550 5050 2000
 $Comp
 L power:GND #PWR0118
 U 1 1 5FD5386E
-P 5300 2850
-F 0 "#PWR0118" H 5300 2600 50  0001 C CNN
-F 1 "GND" H 5305 2677 50  0000 C CNN
-F 2 "" H 5300 2850 50  0001 C CNN
-F 3 "" H 5300 2850 50  0001 C CNN
-	1    5300 2850
+P 5050 2000
+F 0 "#PWR0118" H 5050 1750 50  0001 C CNN
+F 1 "GND" H 5055 1827 50  0000 C CNN
+F 2 "" H 5050 2000 50  0001 C CNN
+F 3 "" H 5050 2000 50  0001 C CNN
+	1    5050 2000
 	1    0    0    -1
 $EndComp
@@
 L power:+5V #PWR0119
 U 1 1 5FD53A6B
-P 5600 1700
-F 0 "#PWR0119" H 5600 1550 50  0001 C CNN
-F 1 "+5V" H 5615 1873 50  0000 C CNN
-F 2 "" H 5600 1700 50  0001 C CNN
-F 3 "" H 5600 1700 50  0001 C CNN
-	1    5600 1700
+P 5350 850
+F 0 "#PWR0119" H 5350 700 50  0001 C CNN
+F 1 "+5V" H 5365 1023 50  0000 C CNN
+F 2 "" H 5350 850 50  0001 C CNN
+F 3 "" H 5350 850 50  0001 C CNN
+	1    5350 850
 	1    0    0    -1
 $EndComp
 Wire Wire Line
-	5200 2400 5200 2650
-Text Label 4800 2550 2    50   ~ 0
+	4950 1550 4950 1800
+Text Label 4550 1700 2    50   ~ 0
 SDA
-Text Label 4800 2650 2    50   ~ 0
+Text Label 4550 1800 2    50   ~ 0
 SCL
 Text Label 1100 3600 2    50   ~ 0
@@
 L EESTN5:CAPAPOL C3
 U 1 1 5FFCE94A
-P 6850 2850
-F 0 "C3" H 6959 2888 40  0000 L CNN
-F 1 "CAPAPOL" H 6959 2812 40  0000 L CNN
-F 2 "EESTN5:CAP_ELEC_SMD_4X5.5" H 6950 2700 30  0001 C CNN
-F 3 "" H 6850 2850 300 0000 C CNN
-	1    6850 2850
+P 5850 1400
+F 0 "C3" H 5959 1438 40  0000 L CNN
+F 1 "CAPAPOL" H 5959 1362 40  0000 L CNN
+F 2 "EESTN5:CAP_ELEC_SMD_4X5.5" H 5950 1250 30  0001 C CNN
+F 3 "" H 5850 1400 300 0000 C CNN
+	1    5850 1400
 	1    0    0    -1
 $EndComp
@@
 L EESTN5:C C4
 U 1 1 5FFCEC57
-P 7150 2850
-F 0 "C4" H 7265 2888 40  0000 L CNN
-F 1 "C" H 7265 2812 40  0000 L CNN
-F 2 "EESTN5:C_1206" H 7188 2700 30  0001 C CNN
-F 3 "" H 7150 2850 60  0000 C CNN
-	1    7150 2850
+P 6150 1400
+F 0 "C4" H 6265 1438 40  0000 L CNN
+F 1 "C" H 6265 1362 40  0000 L CNN
+F 2 "EESTN5:C_1206" H 6188 1250 30  0001 C CNN
+F 3 "" H 6150 1400 60  0000 C CNN
+	1    6150 1400
 	1    0    0    -1
 $EndComp
@@
 L EESTN5:C C5
 U 1 1 5FFCEEDA
-P 7400 2850
-F 0 "C5" H 7515 2888 40  0000 L CNN
-F 1 "C" H 7515 2812 40  0000 L CNN
-F 2 "EESTN5:C_1206" H 7438 2700 30  0001 C CNN
-F 3 "" H 7400 2850 60  0000 C CNN
-	1    7400 2850
+P 6400 1400
+F 0 "C5" H 6515 1438 40  0000 L CNN
+F 1 "C" H 6515 1362 40  0000 L CNN
+F 2 "EESTN5:C_1206" H 6438 1250 30  0001 C CNN
+F 3 "" H 6400 1400 60  0000 C CNN
+	1    6400 1400
 	1    0    0    -1
 $EndComp
@@
 L EESTN5:LED LED1
 U 1 1 5FFCF645
-P 7650 2950
-F 0 "LED1" V 7637 3003 40  0000 L CNN
-F 1 "LED" V 7713 3003 40  0000 L CNN
-F 2 "EESTN5:LED_1206" H 7650 2950 60  0001 C CNN
-F 3 "" H 7650 2950 60  0000 C CNN
-	1    7650 2950
+P 6650 1500
+F 0 "LED1" V 6637 1553 40  0000 L CNN
+F 1 "LED" V 6713 1553 40  0000 L CNN
+F 2 "EESTN5:LED_1206" H 6650 1500 60  0001 C CNN
+F 3 "" H 6650 1500 60  0000 C CNN
+	1    6650 1500
 	0    1    1    0
 $EndComp
@@
 L EESTN5:R R3
 U 1 1 5FFCFAC9
-P 7650 2750
-F 0 "R3" H 7698 2796 50  0000 L CNN
-F 1 "R" H 7698 2705 50  0000 L CNN
-F 2 "EESTN5:R_1206" H 7650 2750 60  0001 C CNN
-F 3 "" H 7650 2750 60  0000 C CNN
-	1    7650 2750
+P 6650 1300
+F 0 "R3" H 6698 1346 50  0000 L CNN
+F 1 "R" H 6698 1255 50  0000 L CNN
+F 2 "EESTN5:R_1206" H 6650 1300 60  0001 C CNN
+F 3 "" H 6650 1300 60  0000 C CNN
+	1    6650 1300
 	1    0    0    -1
 $EndComp
 Wire Wire Line
-	7650 3050 7650 3200
+	6650 1600 6650 1750
 Wire Wire Line
-	7650 3200 7400 3200
+	6650 1750 6400 1750
 Wire Wire Line
-	6850 3200 6850 3050
+	5850 1750 5850 1600
 Wire Wire Line
-	7150 3050 7150 3200
-Connection ~ 7150 3200
+	6150 1600 6150 1750
+Connection ~ 6150 1750
 Wire Wire Line
-	7150 3200 6850 3200
+	6150 1750 5850 1750
 Wire Wire Line
-	7400 3050 7400 3200
-Connection ~ 7400 3200
+	6400 1600 6400 1750
+Connection ~ 6400 1750
 Wire Wire Line
-	7400 3200 7300 3200
+	6400 1750 6300 1750
 Wire Wire Line
-	7300 3200 7300 3350
-Connection ~ 7300 3200
+	6300 1750 6300 1900
+Connection ~ 6300 1750
 Wire Wire Line
-	7300 3200 7150 3200
+	6300 1750 6150 1750
 $Comp
 L power:GND #PWR0134
 U 1 1 6000009B
-P 7300 3350
-F 0 "#PWR0134" H 7300 3100 50  0001 C CNN
-F 1 "GND" H 7305 3177 50  0000 C CNN
-F 2 "" H 7300 3350 50  0001 C CNN
-F 3 "" H 7300 3350 50  0001 C CNN
-	1    7300 3350
+P 6300 1900
+F 0 "#PWR0134" H 6300 1650 50  0001 C CNN
+F 1 "GND" H 6305 1727 50  0000 C CNN
+F 2 "" H 6300 1900 50  0001 C CNN
+F 3 "" H 6300 1900 50  0001 C CNN
+	1    6300 1900
 	1    0    0    -1
 $EndComp
 Wire Wire Line
-	6850 2650 6850 2550
+	5850 1200 5850 1100
 Wire Wire Line
-	7650 2550 7650 2650
+	6650 1100 6650 1200
 Wire Wire Line
-	6850 2550 7150 2550
+	5850 1100 6150 1100
 Wire Wire Line
-	7250 2550 7250 2450
-Connection ~ 7250 2550
+	6250 1100 6250 1000
+Connection ~ 6250 1100
 Wire Wire Line
-	7250 2550 7400 2550
+	6250 1100 6400 1100
 $Comp
 L power:+5V #PWR0135
 U 1 1 6001506C
-P 7250 2450
-F 0 "#PWR0135" H 7250 2300 50  0001 C CNN
-F 1 "+5V" H 7265 2623 50  0000 C CNN
-F 2 "" H 7250 2450 50  0001 C CNN
-F 3 "" H 7250 2450 50  0001 C CNN
-	1    7250 2450
+P 6250 1000
+F 0 "#PWR0135" H 6250 850 50  0001 C CNN
+F 1 "+5V" H 6265 1173 50  0000 C CNN
+F 2 "" H 6250 1000 50  0001 C CNN
+F 3 "" H 6250 1000 50  0001 C CNN
+	1    6250 1000
 	1    0    0    -1
 $EndComp
 Wire Wire Line
-	7150 2550 7150 2650
-Connection ~ 7150 2550
+	6150 1100 6150 1200
+Connection ~ 6150 1100
 Wire Wire Line
-	7150 2550 7250 2550
+	6150 1100 6250 1100
 Wire Wire Line
-	7400 2650 7400 2550
-Connection ~ 7400 2550
+	6400 1200 6400 1100
+Connection ~ 6400 1100
 Wire Wire Line
-	7400 2550 7650 2550
+	6400 1100 6650 1100
 Entry Wire Line
 	8450 5450 8550 5550
@@
 $EndComp
 Wire Wire Line
-	7650 2850 7650 2900
+	6650 1400 6650 1450
 $Comp
 L EESTN5:LM1117-SOT U4
